File: motor-controller/motor-controller.kicad_pcb (KiCad board)
At the start: 2 copper layers, 40 x 50 mm, 60 parts, among them J1 Motor0, J2 Motor1, J3 BATT, J4 MCU, Q1 IRFZ44, Q10 IRFZ44, Q11 IRFZ44, Q12 IRFZ44, Q2 IRFZ44, Q3 IRFZ44, Q4 IRFZ44, Q5 VN2222L, Q6 VN2222L, Q7 VN2222L, Q8 VN2222L, Q9 IRFZ44, U1 MCT6, U2 LT1161, U3 MCT6

Commit message: Update PWM signal selection to avoid an accidental resistor divider
Parts:
- removed H4: M4_PTH, MountingHole:MountingHole_4.3mm_M4_Pad
- added C11: 100nF, Capacitor_THT:C_Disc_D3.0mm_W2.0mm_P2.50mm, F.Cu at (54.0, 54.2)
- added C13: 100nF, Capacitor_THT:C_Disc_D3.0mm_W2.0mm_P2.50mm, F.Cu at (120.3, 68.6)
- added C14: 100nF, Capacitor_THT:C_Disc_D3.0mm_W2.0mm_P2.50mm, F.Cu at (140.3, 71.1)
- added JP1: Motor0_FOW, Jumper:SolderJumper-3_P1.3mm_Bridged12_RoundedPad1.0x1.5mm, B.Cu at (59.1, 43.5)
- added JP2: MOTOR0_REV, Jumper:SolderJumper-3_P1.3mm_Bridged12_RoundedPad1.0x1.5mm, B.Cu at (59.1, 47.4)
- added JP3: MOTOR1_FOW, Jumper:SolderJumper-3_P1.3mm_Bridged12_RoundedPad1.0x1.5mm, B.Cu at (59.1, 51.2)
- added JP4: MOTOR1_REV, Jumper:SolderJumper-3_P1.3mm_Bridged12_RoundedPad1.0x1.5mm, B.Cu at (59.1, 55.1)
- added Q13: 2N3904, Package_TO_SOT_THT:TO-92_Inline, F.Cu at (136.2, 59.7)
- added Q14: VN2222L, Package_TO_SOT_THT:TO-92_Inline, F.Cu at (136.2, 65.4)
- added Q15: IRFZ44, Package_TO_SOT_THT:TO-220-3_Vertical, F.Cu at (142.2, 62.9)
- added Q16: IRFZ44, Package_TO_SOT_THT:TO-220-3_Vertical, F.Cu at (142.2, 78.7)
- added Q17: 2N3904, Package_TO_SOT_THT:TO-92_Inline, F.Cu at (136.9, 79.4)
- added Q18: VN2222L, Package_TO_SOT_THT:TO-92_Inline, F.Cu at (136.9, 73.7)
- added R10: 100k, Resistor_THT:R_Axial_DIN0309_L9.0mm_D3.2mm_P12.70mm_Horizontal, F.Cu at (135.9, 50.8)
- added R11: 10k, Resistor_THT:R_Axial_DIN0309_L9.0mm_D3.2mm_P12.70mm_Horizontal, F.Cu at (136.5, 88.9)
- added R12: 100k, Resistor_THT:R_Axial_DIN0309_L9.0mm_D3.2mm_P12.70mm_Horizontal, F.Cu at (136.5, 92.7)
- added R13: 330R, Resistor_THT:R_Axial_DIN0309_L9.0mm_D3.2mm_P12.70mm_Horizontal, F.Cu at (70.9, 46.1)
- added R14: 1k, Resistor_THT:R_Axial_DIN0309_L9.0mm_D3.2mm_P12.70mm_Horizontal, F.Cu at (70.9, 50.9)
- added R15: 330R, Resistor_THT:R_Axial_DIN0309_L9.0mm_D3.2mm_P12.70mm_Horizontal, F.Cu at (70.9, 55.6)
- added R16: 1k, Resistor_THT:R_Axial_DIN0309_L9.0mm_D3.2mm_P12.70mm_Horizontal, F.Cu at (70.9, 60.4)
- added R17: 330R, Resistor_THT:R_Axial_DIN0309_L9.0mm_D3.2mm_P12.70mm_Horizontal, F.Cu at (70.9, 25.1)
- added R18: 1k, Resistor_THT:R_Axial_DIN0309_L9.0mm_D3.2mm_P12.70mm_Horizontal, F.Cu at (70.9, 29.9)
- added R19: 330R, Resistor_THT:R_Axial_DIN0309_L9.0mm_D3.2mm_P12.70mm_Horizontal, F.Cu at (70.9, 34.6)
- added R20: 1k, Resistor_THT:R_Axial_DIN0309_L9.0mm_D3.2mm_P12.70mm_Horizontal, F.Cu at (70.9, 39.4)
- added R9: 10k, Resistor_THT:R_Axial_DIN0309_L9.0mm_D3.2mm_P12.70mm_Horizontal, F.Cu at (135.9, 47.0)
- C3, C4, C6: value 100nF -> 10nF
- C5: value 47uF -> 10nF; footprint Capacitor_THT:CP_Radial_D5.0mm_P2.00mm -> Capacitor_THT:C_Disc_D3.0mm_W2.0mm_P2.50mm
- C7: value 100nF -> 47uF; footprint Capacitor_THT:C_Disc_D3.0mm_W2.0mm_P2.50mm -> Capacitor_THT:CP_Radial_D5.0mm_P2.00mm
- H1, H2, H3: value M4_PTH -> M3_PTH; footprint MountingHole:MountingHole_4.3mm_M4_Pad -> MountingHole:MountingHole_3.2mm_M3_Pad
- J1, J2, J3: footprint TerminalBlock:TerminalBlock_MaiXu_MX126-5.0-02P_1x02_P5.00mm -> Connector_JST:JST_XH_B2B-XH-A_1x02_P2.50mm_Vertical
- J4: footprint TerminalBlock:TerminalBlock_Xinya_XY308-2.54-5P_1x05_P2.54mm_Horizontal -> Connector_JST:JST_XH_B5B-XH-A_1x05_P2.50mm_Vertical
- Q1, Q2, Q9: value IRFZ44 -> 2N3904; footprint Package_TO_SOT_THT:TO-220-3_Vertical -> Package_TO_SOT_THT:TO-92_Inline
- Q10: value IRFZ44 -> VN2222L; footprint Package_TO_SOT_THT:TO-220-3_Vertical -> Package_TO_SOT_THT:TO-92_Inline
- Q5: value VN2222L -> 2N3904
- Q7, Q8: value VN2222L -> IRFZ44; footprint Package_TO_SOT_THT:TO-92_Inline -> Package_TO_SOT_THT:TO-220-3_Vertical
- R1, R5: value 330R -> 10k
- R2, R6: value 330R -> 100k
- R3, R7: value 1k -> 10k
- R4, R8: value 1k -> 100k
- TP1: value Gate.0+ -> Motor0.+; moved to B.Cu
- TP10: value PwrCtrl.0- -> Motor0.REV_GATE; moved to B.Cu
- TP11: value PwrCtrl.1+ -> Motor1.FOW_GATE; moved to B.Cu
- TP12: value PwrCtrl.1- -> Motor1.REV_GATE; moved to B.Cu
- TP13: value Ctrl.0+ -> Motor1.+; moved to B.Cu
- TP14: value Ctrl.0- -> Motor1.-; moved to B.Cu
- TP15: value Ctrl.1+ -> MCU.PWM1; moved to B.Cu
- TP16: value Ctrl.1- -> MCU.DIR1; moved to B.Cu
- TP17: value GND -> BATT; moved to B.Cu
- TP18: moved to B.Cu
- TP19: value BATT -> MCU_GND; moved to B.Cu
- TP2: value Gate.0- -> MCU.PWM0; moved to B.Cu
- TP3: value Gate.1+ -> Motor0.-; moved to B.Cu
- TP4: value Gate.1- -> MCU.DIR0; moved to B.Cu
- TP5: value Motor.0+ -> Motor0.~{DIR}; moved to B.Cu
- TP6: value Motor.0- -> Motor0.DIR; moved to B.Cu
- TP7: value Motor.1+ -> Motor0.FOW_GATE; moved to B.Cu
- TP8: value Motor.1- -> Motor1.~{DIR}; moved to B.Cu
- TP9: value PwrCtrl.0+ -> Motor1.DIR; moved to B.Cu
- U1: value MCT6 -> LT1161; footprint Package_DIP:DIP-8_W7.62mm_LongPads -> Package_DIP:DIP-20_W7.62mm_LongPads
- U2: value LT1161 -> MCT6; footprint Package_DIP:DIP-20_W7.62mm_LongPads -> Package_DIP:DIP-8_W7.62mm_LongPads
- moved Q2 225.1 mm to (27.7, 58.8), turned to 0 degrees
- moved C10 198.0 mm to (54.0, 50.6), turned to 0 degrees
- moved Q1 157.2 mm to (112.4, 108.0), turned to 0 degrees
- moved Q3 149.3 mm to (113.3, 85.1), turned to 0 degrees
- moved Q4 148.3 mm to (113.3, 56.5), turned to 0 degrees
- moved Q10 148.0 mm to (124.5, 73.7)
- moved H3 135.9 mm to (145.4, 127.0)
- moved Q6 126.6 mm to (123.7, 65.4), turned to -90 degrees
- moved C4 125.8 mm to (126.4, 108.0), turned to 180 degrees
- moved Q5 124.8 mm to (123.7, 59.7), turned to -90 degrees
- moved H2 119.9 mm to (114.9, 127.0)
- moved J2 116.2 mm to (144.8, 71.1)
- moved J1 114.6 mm to (115.8, 68.6)
- moved H1 114.0 mm to (130.2, 49.5)
- moved U2 113.7 mm to (113.0, 120.7), turned to 90 degrees
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Connections:
- C1 pad 2: GND -> GNDPWR
- C10 pad 1: /H-Bridge 1/MOTOR+ -> Net-(C10-Pad1)
- C10 pad 2: /H-Bridge 1/MOTOR- -> GND
- C2 pad 2: GND -> GNDPWR
- C3 pad 1: +BATT -> Net-(U1-T1)
- C3 pad 2: GND -> GNDPWR
- C4 pad 1: /H-Bridge 0/MOTOR+ -> Net-(U1-T2)
- C4 pad 2: /H-Bridge 0/MOTOR- -> GNDPWR
- C5 pad 1: +BATT -> Net-(U1-T3)
- C5 pad 2: GND -> GNDPWR
- C6 pad 1: Net-(C6-Pad1) -> Net-(U1-T4)
- C6 pad 2: GND -> GNDPWR
- C7 pad 1: Net-(C7-Pad1) -> +BATT
- C7 pad 2: GND -> GNDPWR
- C8 pad 1: Net-(C8-Pad1) -> +BATT
- C8 pad 2: GND -> GNDPWR
- C9 pad 2: GND -> GNDPWR
- H1 pad 1: Net-(C6-Pad1) -> Net-(C9-Pad1)
- H2 pad 1: Net-(C7-Pad1) -> Net-(C10-Pad1)
- H3 pad 1: Net-(C8-Pad1) -> Net-(C11-Pad1)
- J3 pad 1: GND -> GNDPWR
- J4 pad 2: /Ctrl.1- -> /MCU.DIR1
- J4 pad 3: /Ctrl.1+ -> /MCU.PWM1
- J4 pad 4: /Ctrl.0- -> /MCU.DIR0
- J4 pad 5: /Ctrl.0+ -> /MCU.PWM0
- Q1 pad 1: /Gate.1+ -> GNDPWR
- Q1 pad 2: +BATT -> Net-(Q1-B)
- Q1 pad 3: /H-Bridge 1/MOTOR+ -> /Motor0.~{DIR}
- Q10 pad 1: /Gate.0- -> /H-Bridge 0/FOW_LOW_GATE
- Q10 pad 2: /H-Bridge 0/MOTOR+ -> /Motor0.DIR
- Q10 pad 3: GND -> GNDPWR
- Q11 pad 1: /Gate.0- -> /H-Bridge 1/FOW_HIGH_GATE
- Q11 pad 3: /H-Bridge 0/MOTOR- -> /H-Bridge 1/MOTOR+
- Q12 pad 1: /Gate.0+ -> /H-Bridge 1/REV_HIGH_GATE
- Q12 pad 2: /H-Bridge 0/MOTOR- -> +BATT
- Q12 pad 3: GND -> /H-Bridge 1/MOTOR-
- Q2 pad 1: /Gate.1- -> GNDPWR
- Q2 pad 2: +BATT -> Net-(Q2-B)
- Q2 pad 3: /H-Bridge 1/MOTOR- -> /Motor1.~{DIR}
- Q3 pad 1: /Gate.1- -> /H-Bridge 0/FOW_HIGH_GATE
- Q3 pad 2: /H-Bridge 1/MOTOR+ -> +BATT
- Q3 pad 3: GND -> /H-Bridge 0/MOTOR+
- Q4 pad 1: /Gate.1+ -> /H-Bridge 0/REV_HIGH_GATE
- Q4 pad 2: /H-Bridge 1/MOTOR- -> +BATT
- Q4 pad 3: GND -> /H-Bridge 0/MOTOR-
- Q5 pad 1: /Gate.1+ -> GNDPWR
- Q5 pad 2: /Gate.1- -> Net-(Q5-B)
- Q5 pad 3: GND -> /H-Bridge 0/REV_LOW_GATE
- Q6 pad 1: /Gate.1- -> /H-Bridge 0/REV_LOW_GATE
- Q6 pad 2: /Gate.1+ -> /Motor0.~{DIR}
- Q6 pad 3: GND -> GNDPWR
- Q7 pad 1: /Gate.0+ -> /H-Bridge 0/REV_LOW_GATE
- Q7 pad 2: /Gate.0- -> /H-Bridge 0/MOTOR+
- Q7 pad 3: GND -> GNDPWR
- Q8 pad 1: /Gate.0- -> /H-Bridge 0/FOW_LOW_GATE
- Q8 pad 2: /Gate.0+ -> /H-Bridge 0/MOTOR-
- Q8 pad 3: GND -> GNDPWR
- Q9 pad 1: /Gate.0+ -> GNDPWR
- Q9 pad 2: +BATT -> Net-(Q9-B)
- Q9 pad 3: /H-Bridge 0/MOTOR+ -> /H-Bridge 0/FOW_LOW_GATE
- R1 pad 1: /Ctrl.0+ -> +BATT
- R1 pad 2: Net-(R1-Pad2) -> /Motor0.~{DIR}
- R2 pad 1: /Ctrl.0- -> /Motor0.DIR
- R2 pad 2: Net-(R2-Pad2) -> Net-(Q1-B)
- R3 pad 1: GND -> +BATT
- R3 pad 2: /PwrCtrl.0- -> /Motor1.~{DIR}
- R4 pad 1: GND -> /Motor1.DIR
- R4 pad 2: /PwrCtrl.0+ -> Net-(Q2-B)
- R5 pad 1: /Ctrl.1+ -> +BATT
- R5 pad 2: Net-(R5-Pad2) -> /H-Bridge 0/REV_LOW_GATE
- R6 pad 1: /Ctrl.1- -> /PWM0
- R6 pad 2: Net-(R6-Pad2) -> Net-(Q5-B)
- R7 pad 1: GND -> +BATT
- R7 pad 2: /PwrCtrl.1+ -> /H-Bridge 0/FOW_LOW_GATE
- R8 pad 1: GND -> /PWM0
- R8 pad 2: /PwrCtrl.1- -> Net-(Q9-B)
- TP1 pad 1: /Gate.0+ -> /H-Bridge 0/MOTOR+
- TP10 pad 1: /PwrCtrl.0- -> /H-Bridge 0/REV_HIGH_GATE
- TP11 pad 1: /PwrCtrl.1+ -> /H-Bridge 1/FOW_HIGH_GATE
- TP12 pad 1: /PwrCtrl.1- -> /H-Bridge 1/REV_HIGH_GATE
- TP13 pad 1: /Ctrl.0+ -> /H-Bridge 1/MOTOR+
- TP14 pad 1: /Ctrl.0- -> /H-Bridge 1/MOTOR-
- TP15 pad 1: /Ctrl.1+ -> /MCU.PWM1
- TP16 pad 1: /Ctrl.1- -> /MCU.DIR1
- TP17 pad 1: GND -> +BATT
- TP18 pad 1: GND -> GNDPWR
- TP19 pad 1: +BATT -> GND
- TP2 pad 1: /Gate.0- -> /MCU.PWM0
- TP3 pad 1: /Gate.1+ -> /H-Bridge 0/MOTOR-
- TP4 pad 1: /Gate.1- -> /MCU.DIR0
- TP5 pad 1: /H-Bridge 0/MOTOR+ -> /Motor0.~{DIR}
- TP6 pad 1: /H-Bridge 0/MOTOR- -> /Motor0.DIR
- TP7 pad 1: /H-Bridge 1/MOTOR+ -> /H-Bridge 0/FOW_HIGH_GATE
- TP8 pad 1: /H-Bridge 1/MOTOR- -> /Motor1.~{DIR}
- TP9 pad 1: /PwrCtrl.0+ -> /Motor1.DIR
- U1 pad 1: Net-(R1-Pad2) -> GNDPWR
- U1 pad 2: GND -> Net-(U1-T1)
- U1 pad 3: GND -> /Motor0.~{DIR}
- U1 pad 4: Net-(R2-Pad2) -> Net-(U1-T2)
- U1 pad 5: /PwrCtrl.0- -> /Motor0.DIR
- U1 pad 6: +BATT -> Net-(U1-T3)
- U1 pad 7: +BATT -> /Motor1.~{DIR}
- U1 pad 8: /PwrCtrl.0+ -> Net-(U1-T4)
- U2 pad 1: GND -> Net-(R13-Pad2)
- U2 pad 2: unconnected-(U2-T1-Pad2) -> GND
- U2 pad 3: /PwrCtrl.0+ -> GND
- U2 pad 4: unconnected-(U2-T2-Pad4) -> Net-(R15-Pad2)
- U2 pad 5: /PwrCtrl.0- -> /Motor0.DIR
- U2 pad 6: unconnected-(U2-T3-Pad6) -> +BATT
- U2 pad 7: /PwrCtrl.1+ -> +BATT
- U2 pad 8: unconnected-(U2-T4-Pad8) -> /Motor0.PWM
- U3 pad 1: Net-(R5-Pad2) -> Net-(R17-Pad2)
- U3 pad 4: Net-(R6-Pad2) -> Net-(R19-Pad2)
- U3 pad 5: /PwrCtrl.1- -> /Motor1.DIR
- U3 pad 8: /PwrCtrl.1+ -> /Motor1.PWM
Other:
- board size 40 x 50 mm -> 40.6 x 87.6 mm

Commit message: Finish layout
Parts:
- removed TP1: Motor0.+, TestPoint:TestPoint_Pad_1.5x1.5mm
- removed TP13: Motor1.+, TestPoint:TestPoint_Pad_1.5x1.5mm
- removed TP14: Motor1.-, TestPoint:TestPoint_Pad_1.5x1.5mm
- removed TP15: MCU.PWM1, TestPoint:TestPoint_Pad_1.5x1.5mm
- removed TP16: MCU.DIR1, TestPoint:TestPoint_Pad_1.5x1.5mm
- removed TP2: MCU.PWM0, TestPoint:TestPoint_Pad_1.5x1.5mm
- removed TP3: Motor0.-, TestPoint:TestPoint_Pad_1.5x1.5mm
- removed TP4: MCU.DIR0, TestPoint:TestPoint_Pad_1.5x1.5mm
- added C12: 100nF, Capacitor_THT:C_Disc_D3.0mm_W2.0mm_P2.50mm, F.Cu at (128.9, 76.2)
- R14, R16, R18, R20: value 1k -> 10k
- moved R1 141.8 mm to (128.3, 135.3), turned to 90 degrees
- moved R3 137.2 mm to (132.1, 135.3), turned to 90 degrees
- moved TP19 135.5 mm to (139.1, 141.0)
- moved R17 124.6 mm to (135.9, 131.4)
- moved Q2 124.3 mm to (136.5, 118.7), turned to -90 degrees
- moved C11 122.7 mm to (146.1, 135.3)
- moved R2 118.3 mm to (128.3, 107.3), turned to -90 degrees
- moved R4 115.3 mm to (132.1, 107.3), turned to -90 degrees
- moved R19 113.4 mm to (135.9, 127.6)
- moved TP6 112.9 mm to (128.3, 115.6)
- moved U3 112.7 mm to (141.0, 123.8), turned to 90 degrees
- moved TP9 106.9 mm to (132.1, 115.6)
- moved TP8 106.3 mm to (132.1, 111.1)
- moved C10 103.9 mm to (114.3, 135.3), turned to 180 degrees
- moved R18 102.1 mm to (135.9, 108.6)
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Connections:
- Q13 pad 1: GNDPWR -> /H-Bridge 1/REV_LOW_GATE
- Q13 pad 3: /H-Bridge 1/REV_LOW_GATE -> +BATT
- Q17 pad 1: GNDPWR -> /H-Bridge 1/FOW_LOW_GATE
- Q17 pad 3: /H-Bridge 1/FOW_LOW_GATE -> +BATT
- Q5 pad 1: GNDPWR -> /H-Bridge 0/REV_LOW_GATE
- Q5 pad 3: /H-Bridge 0/REV_LOW_GATE -> +BATT
- Q9 pad 1: GNDPWR -> /H-Bridge 0/FOW_LOW_GATE
- Q9 pad 3: /H-Bridge 0/FOW_LOW_GATE -> +BATT
- R11 pad 1: +BATT -> /H-Bridge 1/FOW_LOW_GATE
- R11 pad 2: /H-Bridge 1/FOW_LOW_GATE -> GNDPWR
- R5 pad 1: +BATT -> /H-Bridge 0/REV_LOW_GATE
- R5 pad 2: /H-Bridge 0/REV_LOW_GATE -> GNDPWR
- R7 pad 1: +BATT -> /H-Bridge 0/FOW_LOW_GATE
- R7 pad 2: /H-Bridge 0/FOW_LOW_GATE -> GNDPWR
- R9 pad 1: +BATT -> /H-Bridge 1/REV_LOW_GATE
- R9 pad 2: /H-Bridge 1/REV_LOW_GATE -> GNDPWR
Routing:
- net +BATT: track 0.00 -> 94.7 mm, vias 0 -> 5
- net /Motor1.DIR: track 0.00 -> 78.3 mm, vias 0 -> 1
- net /Motor0.~{DIR}: track 0.00 -> 73.3 mm, vias 0 -> 3
- net /Motor0.DIR: track 0.00 -> 72.9 mm, vias 0 -> 3
- net /Motor1.~{DIR}: track 0.00 -> 64.6 mm, vias 0 -> 2
- net /H-Bridge 1/REV_HIGH_GATE: track 0.00 -> 47.0 mm
- net /PWM0: track 0.00 -> 44.4 mm
- net /PWM1: track 0.00 -> 44.1 mm
- net /H-Bridge 1/REV_LOW_GATE: track 0.00 -> 43.9 mm
- net /H-Bridge 0/FOW_HIGH_GATE: track 0.00 -> 41.1 mm, vias 0 -> 1
- net /H-Bridge 1/FOW_LOW_GATE: track 0.00 -> 36.4 mm
- net Net-(Q9-B): track 0.00 -> 28.0 mm
- net /H-Bridge 0/FOW_LOW_GATE: track 0.00 -> 26.8 mm
- net /H-Bridge 1/FOW_HIGH_GATE: track 0.00 -> 26.5 mm, vias 0 -> 1
- net /H-Bridge 0/REV_LOW_GATE: track 0.00 -> 25.0 mm
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- added copper zone on F.Cu, net +BATT
- added copper zone on B.Cu, net GND
- added copper zone on F.Cu, net GND
- added copper zone on B.Cu, net GNDPWR
- added copper zone on F.Cu, net GNDPWR
Other:
- board size 40.6 x 87.6 mm -> 40.9 x 101.2 mm

Commit message: Generate schematic pdf
Parts:
- added REF**: , GS_Virtual:ENPH253_Logo_Small, F.Cu at (130.2, 84.6)
- added REF**: OSHW-Logo_7.5x8mm_SilkScreen, Symbol:OSHW-Logo_7.5x8mm_SilkScreen, B.Cu at (142.2, 50.0)
- moved C6 3.18 mm to (148.0, 101.6)
- moved C3 3.17 mm to (112.4, 101.6)
- moved C5 2.62 mm to (148.0, 99.0), turned to 90 degrees
- moved C4 2.54 mm to (112.4, 99.1), turned to 90 degrees
- moved J4 0.76 mm to (135.2, 140.2)
- moved H2 0.13 mm to (114.3, 141.1)
- moved H3 0.13 mm to (146.1, 141.1)
- renumbered JP2 to DIR0, TP6 to DIR0, JP4 to DIR1, TP9 to DIR1, TP7 to M0.Fow_Gate, TP10 to M0.Rev_Gate, TP11 to M1.Fow_Gate, TP12 to M1.Rev_Gate, TP19 to MCU.GND, JP1 to ~{DIR0}, TP5 to ~{DIR0}, JP3 to ~{DIR1}, TP8 to ~{DIR1}
Routing:
- net Net-(U1-T4): track 9.29 -> 12.5 mm
- net Net-(U1-T1): track 6.77 -> 9.94 mm
- net /MCU.DIR0: track 11.5 -> 10.1 mm
- net /MCU.PWM1: track 12.1 -> 11.1 mm
- net /MCU.PWM0: track 14.6 -> 13.8 mm
- net /MCU.DIR1: track 15.6 -> 14.9 mm
- net /H-Bridge 0/FOW_LOW_GATE: track 26.8 -> 26.2 mm
- net /H-Bridge 1/FOW_HIGH_GATE: track 26.5 -> 25.9 mm
Other:
- board size 40.9 x 101.2 mm -> 40.9 x 101.5 mm
- board text added: "+"
- board text added: "-"
- board text added: "0.DIR"
- board text added: "0.PWM"
- board text added: "Battery configuration: 4S"
- board text added: "GND"
- board text added: "H-Bridge"
- board text added: "Jump to enable extra shoot through protection"
- board text added: "Rev A"
