File: dual-h-bridge/dual-h-bridge.kicad_sch (KiCad schematic)
At the start: 42 parts, among them J1 Motor0, J2 Motor1, J3 BATT, J4 MCU, Q1 2N3904, Q2 2N3904, U1 LT1161

Commit message: Change to new connector standard
Parts:
- J4: symbol Connector:Conn_01x05_Socket -> Connector:Conn_01x06_Socket
Connections:
- no-connect marks 0 -> 1
Changed lines of the file:
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@@
 		(color 0 0 0 0)
+	)
+	(no_connect
+		(at 39.37 153.67)
 	)
 	(wire
@@
 	)
 	(symbol
-		(lib_id "Connector:Conn_01x05_Socket")
+		(lib_id "Connector:Conn_01x06_Socket")
 		(at 34.29 161.29 180)
 		(unit 1)
@@
 		(dnp no)
 		(property "Reference" "J4"
-			(at 30.988 160.02 0)
+			(at 30.988 158.75 0)
 			(effects
 				(font
@@
 		)
 		(property "Value" "MCU"
-			(at 30.988 162.56 0)
+			(at 30.988 161.29 0)
 			(effects
 				(font
@@
 			)
 		)
-		(property "Description" "Generic connector, single row, 01x05, script generated"
+		(property "Description" "Generic connector, single row, 01x06, script generated"
 			(at 34.29 161.29 0)
 			(effects
@@
 		(pin "5"
 		)
+		(pin "6"
+		)
 		(instances
