File: dual-h-bridge/dual-h-bridge.kicad_pcb (KiCad board)
At the start: 2 copper layers, 40.9 x 101.5 mm, 78 parts, among them J1 Motor0, J2 Motor1, J3 BATT, J4 MCU, Q1 2N3904, Q10 VN2222L, Q11 IRFZ44, Q12 IRFZ44, Q13 2N3904, Q14 VN2222L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

Commit message: Update silkscreen
Parts:
- added REF**: KiCad-Logo2_6mm_SilkScreen, Symbol:KiCad-Logo2_6mm_SilkScreen, B.Cu at (212.7, 79.4)
- added REF**: OSHW-Logo_7.5x8mm_SilkScreen, Symbol:OSHW-Logo_7.5x8mm_SilkScreen, B.Cu at (224.8, 46.4)
Other:
- board text added: "v2.0.1"
- board text removed: "v2.0.0"
